File: hardware/bicyclelab-charger-3.brd (EAGLE design)
At the start: 87 x 27.9 mm, 45 parts, among them IC1 LDO-5V-0.5A, IC2 TINY24/44/84-SSU, Q1 BC817-16SMD, Q2 FDP5800

Commit message: implement code for tiny and arduino, check Makefile.p328
Parts:
- moved R7 62.9 mm to (48.6, 26.4), turned to 180 degrees
Routing:
- net N$4: track 0.00 -> 2.64 mm
- net N$1: track 64.0 -> 62.5 mm
Changed lines of the file:
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@@
 <element name="R6" library="SparkFun" package="0805" value="1k" x="20.955" y="4.7625" rot="R180"/>
 <element name="VBOOST" library="SparkFun" package="1X01NS" value="" x="52.07" y="15.24"/>
-<element name="R7" library="SparkFun" package="0805" value="47" x="-1.905" y="-11.1125"/>
+<element name="R7" library="SparkFun" package="0805" value="47" x="48.5775" y="26.3525" rot="R180"/>
 </elements>
 <signals>
@@
 <contactref element="IC2" pad="5"/>
 <contactref element="FET" pad="1"/>
-<wire x1="48.5775" y1="25.4" x2="47.9425" y2="26.3525" width="0.4064" layer="1"/>
-<wire x1="47.9425" y1="26.3525" x2="45.72" y2="26.3525" width="0.4064" layer="1"/>
+<wire x1="47.3075" y1="26.3525" x2="45.72" y2="26.3525" width="0.4064" layer="1"/>
 <wire x1="45.72" y1="26.3525" x2="29.5275" y2="26.3525" width="0.4064" layer="16"/>
 <wire x1="29.5275" y1="26.3525" x2="26.3525" y2="23.1775" width="0.4064" layer="16"/>
@@
 <wire x1="8.89" y1="4.7625" x2="9.525" y2="4.7625" width="0.4064" layer="16"/>
 <contactref element="R7" pad="2"/>
-<wire x1="7.5565" y1="4.7625" x2="-1.005" y2="-11.1125" width="0" layer="19" extent="1-1"/>
+<wire x1="47.3075" y1="26.3525" x2="47.6775" y2="26.3525" width="0.6096" layer="1"/>
 </signal>
 <signal name="N$3">
@@
 <contactref element="R7" pad="1"/>
 <contactref element="Q2" pad="B"/>
-<wire x1="-2.805" y1="-11.1125" x2="48.5775" y2="24.13" width="0" layer="19" extent="1-1"/>
+<wire x1="48.5775" y1="24.13" x2="49.53" y2="25.0825" width="0.6096" layer="1"/>
+<wire x1="49.53" y1="25.0825" x2="49.53" y2="26.3" width="0.6096" layer="1"/>
+<wire x1="49.53" y1="26.3" x2="49.4775" y2="26.3525" width="0.6096" layer="1"/>
 </signal>
 </signals>
